Commit message: change name

File: urdf/ur10e_with_lift.ros2_control.xacro (robot description, xacro)
@@ -1,5 +1,5 @@
 <?xml version="1.0"?>
 <robot xmlns:xacro="http://www.ros.org/wiki/xacro">
-  <xacro:macro name="ur10e_with_lift_ros2_control" params="
+  <xacro:macro name="ur_ros2_control" params="
     name
     use_fake_hardware:=false fake_sensor_commands:=false

File: urdf/ur10e_with_lift.urdf.xacro (robot description, xacro)
@@ -2,5 +2,5 @@
 <robot xmlns:xacro="http://wiki.ros.org/xacro" name="$(arg name)">
    <!-- robot name parameter -->
-   <xacro:arg name="name" default="ur10e_with_lift"/>
+   <xacro:arg name="name" default="ur"/>
    <!-- import main macro -->
    <xacro:include filename="$(find ur10e_arm_with_lift)/urdf/ur10e_with_lift_macro.xacro"/>
@@ -110,5 +110,5 @@
     </joint>
    <!-- arm -->
-   <xacro:ur10e_with_lift_robot
+   <xacro:ur_robot
      name="$(arg name)"
      tf_prefix="$(arg tf_prefix)"

File: urdf/ur10e_with_lift_macro.xacro (robot description, xacro)
@@ -3,5 +3,5 @@
   <xacro:include filename="$(find ur_description)/urdf/inc/ur_transmissions.xacro" />
   <xacro:include filename="$(find ur_description)/urdf/inc/ur_common.xacro" />
-  <xacro:macro name="ur10e_with_lift_robot" params="
+  <xacro:macro name="ur_robot" params="
     name
     tf_prefix
@@ -55,5 +55,5 @@
       <xacro:include filename="$(find ur10e_arm_with_lift)/urdf/ur_with_lift.ros2_control.xacro" />
       <!-- ros2 control instance -->
-      <xacro:ur10e_with_lift_ros2_control
+      <xacro:ur_ros2_control
         name="${name}"
         use_fake_hardware="${use_fake_hardware}"

Commit message: test urdf and crontrollers

File: urdf/ur10e_with_lift.ros2_control.xacro (robot description, xacro)
@@ -1,5 +1,5 @@
 <?xml version="1.0"?>
 <robot xmlns:xacro="http://www.ros.org/wiki/xacro">
-  <xacro:macro name="ur_ros2_control" params="
+  <xacro:macro name="ur10e_with_lift_ros2_control" params="
     name
     use_fake_hardware:=false fake_sensor_commands:=false

File: urdf/ur10e_with_lift.urdf.xacro (robot description, xacro)
@@ -2,5 +2,5 @@
 <robot xmlns:xacro="http://wiki.ros.org/xacro" name="$(arg name)">
    <!-- robot name parameter -->
-   <xacro:arg name="name" default="ur"/>
+   <xacro:arg name="name" default="ur10e_with_lift"/>
    <!-- import main macro -->
    <xacro:include filename="$(find ur10e_arm_with_lift)/urdf/ur10e_with_lift_macro.xacro"/>
@@ -77,41 +77,9 @@
      </joint>
    </xacro:if>
-    <!-- Lift Link -->
-    <link name="${tf_prefix}lift_link">
-      <visual>
-        <origin xyz="0 0 0.07" rpy="0 0 0"/>
-        <geometry>
-          <box size="0.50 0.50 0.14"/>
-        </geometry>
-        <material name="lift_grey">
-           <color rgba="0.6 0.6 0.6 1"/>
-        </material>
-      </visual>
-      <collision>
-        <origin xyz="0 0 0.07" rpy="0 0 0"/>
-        <geometry>
-          <box size="0.50 0.50 0.14"/>
-        </geometry>
-      </collision>
-      <inertial>
-        <mass value="33"/>
-        <origin rpy="0 0 0 " xyz="0 0 0.07"/>
-        <inertia ixx="0.1" ixy="0.0" ixz="0.0" iyy="0.1" iyz="0.0" izz="0.1"/>
-      </inertial>
-    </link>
-    <!-- Vertical Prismatic Joint -->
-    <joint name="${tf_prefix}lift_joint" type="prismatic">
-      <parent link="world" />
-      <child link="lift_link" />
-      <origin xyz="0 0 0 " rpy="0 0 0" />
-      <axis xyz="0 0 1" />
-      <limit lower="0.0" upper="1.0" effort="500" velocity="0.5"/>
-      <dynamics damping="0" friction="0"/>
-    </joint>
-   <!-- arm -->
-   <xacro:ur_robot
+   <!-- ur10e arm with lift -->
+   <xacro:ur10e_with_lift_robot
      name="$(arg name)"
      tf_prefix="$(arg tf_prefix)"
-     parent="lift_link"
+     parent="world"
      joint_limits_parameters_file="$(arg joint_limit_params)"
      kinematics_parameters_file="$(arg kinematics_params)"
@@ -148,5 +116,5 @@
      >
      <origin xyz="0 0 0" rpy="0 0 0" />          <!-- position robot in the world -->
-   </xacro:ur_robot>
+   </xacro:ur10e_with_lift_robot>
    <xacro:if value="$(arg sim_gazebo)">
     <!-- Gazebo plugins -->

File: urdf/ur10e_with_lift_macro.xacro (robot description, xacro)
@@ -3,5 +3,5 @@
   <xacro:include filename="$(find ur_description)/urdf/inc/ur_transmissions.xacro" />
   <xacro:include filename="$(find ur_description)/urdf/inc/ur_common.xacro" />
-  <xacro:macro name="ur_robot" params="
+  <xacro:macro name="ur10e_with_lift_robot" params="
     name
     tf_prefix
@@ -53,7 +53,7 @@
     <xacro:if value="${generate_ros2_control_tag}">
       <!-- ros2 control include -->
-      <xacro:include filename="$(find ur10e_arm_with_lift)/urdf/ur_with_lift.ros2_control.xacro" />
+      <xacro:include filename="$(find ur10e_arm_with_lift)/urdf/ur10e_with_lift.ros2_control.xacro" />
       <!-- ros2 control instance -->
-      <xacro:ur_ros2_control
+      <xacro:ur10e_with_lift_ros2_control
         name="${name}"
         use_fake_hardware="${use_fake_hardware}"
@@ -91,4 +91,27 @@
     <!-- Placeholder for ros2_control transmission which don't yet exist -->
     <!-- links -  main serial chain -->
+    <!-- Lift Link -->
+    <link name="${tf_prefix}lift_link">
+      <visual>
+        <origin xyz="0 0 0.07" rpy="0 0 0"/>
+        <geometry>
+          <box size="0.50 0.50 0.14"/>
+        </geometry>
+        <material name="lift_grey">
+           <color rgba="0.6 0.6 0.6 1"/>
+        </material>
+      </visual>
+      <collision>
+        <origin xyz="0 0 0.07" rpy="0 0 0"/>
+        <geometry>
+          <box size="0.50 0.50 0.14"/>
+        </geometry>
+      </collision>
+      <inertial>
+        <mass value="33"/>
+        <origin rpy="0 0 0 " xyz="0 0 0.07"/>
+        <inertia ixx="0.1" ixy="0.0" ixz="0.0" iyy="0.1" iyz="0.0" izz="0.1"/>
+      </inertial>
+    </link>
     <link name="${tf_prefix}base_link"/>
     <link name="${tf_prefix}base_link_inertia">
@@ -273,8 +296,16 @@
       </inertial>
     </link>
+    <!-- Vertical Prismatic Joint -->
+    <joint name="${tf_prefix}lift_joint" type="prismatic">
+      <parent link="${parent}" />
+      <child link="${tf_prefix}lift_link" />
+      <origin xyz="0 0 0 " rpy="0 0 0" />
+      <axis xyz="0 0 1" />
+      <limit lower="0.0" upper="1.0" effort="500" velocity="0.5"/>
+    </joint>
     <!-- base_joint fixes base_link to the environment -->
     <joint name="${tf_prefix}base_joint" type="fixed">
       <origin xyz="0 0 0.15" rpy="0 0 ${pi}" />
-      <parent link="${parent}" />
+      <parent link="${tf_prefix}lift_link" />
       <child link="${tf_prefix}base_link" />
     </joint>
