Commit message: add controllers

File: urdf/ur10e_with_lift.urdf.xacro (robot description, xacro)
@@ -78,12 +78,34 @@
    </xacro:if>
     <!-- Lift Link -->
-    <link name="lift_link"/>
+    <link name="lift_link">
+      <visual>
+        <origin xyz="0 0 0.07" rpy="0 0 0"/>
+        <geometry>
+          <box size="0.50 0.50 0.14"/>
+        </geometry>
+        <material name="lift_grey">
+           <color rgba="0.2 0.2 0.2 1"/>
+        </material>
+      </visual>
+      <collision>
+        <origin xyz="0 0 0.07" rpy="0 0 0"/>
+        <geometry>
+          <box size="0.50 0.50 0.14"/>
+        </geometry>
+      </collision>
+      <inertial>
+        <mass value="33"/>
+        <origin rpy="0 0 0 " xyz="0 0 0.07"/>
+        <inertia ixx="0.1" ixy="0.0" ixz="0.0" iyy="0.1" iyz="0.0" izz="0.1"/>
+      </inertial>
+    </link>
     <!-- Vertical Prismatic Joint -->
     <joint name="lift_joint" type="prismatic">
-        <parent link="world"/>
-        <child link="lift_link"/>
-        <origin xyz="0 0 0" rpy="0 0 0"/>
-        <axis xyz="0 0 1"/>
-        <limit lower="0.0" upper="1.0" effort="500" velocity="0.5"/>
+      <parent link="world" />
+      <child link="lift_link" />
+      <origin xyz="0 0 0 " rpy="0 0 0" />
+      <axis xyz="0 0 1" />
+      <limit lower="0.0" upper="1.0" effort="500" velocity="0.5"/>
+      <dynamics damping="0" friction="0"/>
     </joint>
    <!-- arm -->
@@ -148,3 +170,22 @@
     </gazebo>
   </xacro:if>
+  <!-- <ros2_control name="lift_control" type="system">
+    <hardware>
+      <xacro:if value="${arg sim_gazebo}">
+        <plugin>gazebo_ros2_control/GazeboSystem</plugin>
+      </xacro:if>
+      <xacro:if value="${arg sim_ignition}">
+        <plugin>ign_ros2_control/IgnitionSystem</plugin>
+      </xacro:if>
+    </hardware>
+    <joint name="lift_joint">
+      <command_interface name="position"/>
+      <command_interface name="velocity"/>
+      <state_interface name="position">
+        <param name="initial_value">0.0</param>
+      </state_interface>
+      <state_interface name="velocity"/>
+      <state_interface name="effort"/>
+    </joint>
+  </ros2_control> -->
 </robot>

Commit message: modify controllers

File: urdf/ur10e_with_lift.urdf.xacro (robot description, xacro)
@@ -78,5 +78,5 @@
    </xacro:if>
     <!-- Lift Link -->
-    <link name="lift_link">
+    <link name="${tf_prefix}lift_link">
       <visual>
         <origin xyz="0 0 0.07" rpy="0 0 0"/>
@@ -101,5 +101,5 @@
     </link>
     <!-- Vertical Prismatic Joint -->
-    <joint name="lift_joint" type="prismatic">
+    <joint name="${tf_prefix}lift_joint" type="prismatic">
       <parent link="world" />
       <child link="lift_link" />
@@ -110,5 +110,5 @@
     </joint>
    <!-- arm -->
-   <xacro:ur_robot
+   <xacro:ur10e_with_lift_robot
      name="$(arg name)"
      tf_prefix="$(arg tf_prefix)"
@@ -170,56 +170,3 @@
     </gazebo>
   </xacro:if>
-  <!-- <ros2_control name="lift_control" type="system">
-    <hardware>
-      <xacro:if value="$(arg sim_gazebo)">
-        <plugin>gazebo_ros2_control/GazeboSystem</plugin>
-      </xacro:if>
-      <xacro:if value="$(arg sim_ignition)">
-        <plugin>ign_ros2_control/IgnitionSystem</plugin>
-      </xacro:if>
-      <xacro:if value="$(arg use_fake_hardware)">
-        <plugin>mock_components/GenericSystem</plugin>
-        <param name="fake_sensor_commands">${fake_sensor_commands}</param>
-        <param name="state_following_offset">0.0</param>
-        <param name="calculate_dynamics">true</param>
-      </xacro:if>
-      <xacro:unless value="$(arg use_fake_hardware or arg sim_gazebo or arg sim_ignition)">
-        <plugin>ur_robot_driver/URPositionHardwareInterface</plugin>
-        <param name="robot_ip">$(arg robot_ip)</param>
-        <param name="script_filename">$(arg script_filename)</param>
-        <param name="output_recipe_filename">$(arg output_recipe_filename)</param>
-        <param name="input_recipe_filename">$(arg input_recipe_filename)</param>
-        <param name="headless_mode">$(arg headless_mode)</param>
-        <param name="reverse_port">$(arg reverse_port)</param>
-        <param name="script_sender_port">$(arg script_sender_port)</param>
-        <param name="reverse_ip">$(arg reverse_ip)</param>
-        <param name="script_command_port">$(arg script_command_port)</param>
-        <param name="trajectory_port">$(arg trajectory_port)</param>
-        <param name="tf_prefix">$(arg tf_prefix)</param>
-        <param name="non_blocking_read">$(arg non_blocking_read)</param>
-        <param name="servoj_gain">2000</param>
-        <param name="servoj_lookahead_time">0.03</param>
-        <param name="use_tool_communication">$(arg use_tool_communication)</param>
-        <param name="kinematics/hash">$(arg hash_kinematics)</param>
-        <param name="tool_voltage">$(arg tool_voltage)</param>
-        <param name="tool_parity">$(arg tool_parity)</param>
-        <param name="tool_baud_rate">$(arg tool_baud_rate)</param>
-        <param name="tool_stop_bits">$(arg tool_stop_bits)</param>
-        <param name="tool_rx_idle_chars">$(arg tool_rx_idle_chars)</param>
-        <param name="tool_tx_idle_chars">$(arg tool_tx_idle_chars)</param>
-        <param name="tool_device_name">$(arg tool_device_name)</param>
-        <param name="tool_tcp_port">$(arg tool_tcp_port)</param>
-        <param name="keep_alive_count">$(arg keep_alive_count)</param>
-      </xacro:unless>
-    </hardware>
-    <joint name="lift_joint">
-      <command_interface name="position"/>
-      <command_interface name="velocity"/>
-      <state_interface name="position">
-        <param name="initial_value">0.0</param>
-      </state_interface>
-      <state_interface name="velocity"/>
-      <state_interface name="effort"/>
-    </joint>
-  </ros2_control> -->
 </robot>

File: urdf/ur10e_with_lift_macro.xacro (robot description, xacro)
@@ -3,5 +3,5 @@
   <xacro:include filename="$(find ur_description)/urdf/inc/ur_transmissions.xacro" />
   <xacro:include filename="$(find ur_description)/urdf/inc/ur_common.xacro" />
-  <xacro:macro name="ur_robot" params="
+  <xacro:macro name="ur10e_with_lift_robot" params="
     name
     tf_prefix
@@ -53,7 +53,7 @@
     <xacro:if value="${generate_ros2_control_tag}">
       <!-- ros2 control include -->
-      <xacro:include filename="$(find ur_description)/urdf/ur.ros2_control.xacro" />
+      <xacro:include filename="$(find ur10e_arm_with_lift)/urdf/ur_with_lift.ros2_control.xacro" />
       <!-- ros2 control instance -->
-      <xacro:ur_ros2_control
+      <xacro:ur10e_with_lift_ros2_control
         name="${name}"
         use_fake_hardware="${use_fake_hardware}"

Commit message: change name

File: urdf/ur10e_with_lift.urdf.xacro (robot description, xacro)
@@ -2,5 +2,5 @@
 <robot xmlns:xacro="http://wiki.ros.org/xacro" name="$(arg name)">
    <!-- robot name parameter -->
-   <xacro:arg name="name" default="ur10e_with_lift"/>
+   <xacro:arg name="name" default="ur"/>
    <!-- import main macro -->
    <xacro:include filename="$(find ur10e_arm_with_lift)/urdf/ur10e_with_lift_macro.xacro"/>
@@ -78,5 +78,5 @@
    </xacro:if>
    <!-- ur10e arm with lift -->
-   <xacro:ur10e_with_lift_robot
+   <xacro:ur_robot
      name="$(arg name)"
      tf_prefix="$(arg tf_prefix)"
@@ -116,5 +116,5 @@
      >
      <origin xyz="0 0 0" rpy="0 0 0" />          <!-- position robot in the world -->
-   </xacro:ur10e_with_lift_robot>
+   </xacro:ur_robot>
    <xacro:if value="$(arg sim_gazebo)">
     <!-- Gazebo plugins -->

File: urdf/ur10e_with_lift_macro.xacro (robot description, xacro)
@@ -3,5 +3,5 @@
   <xacro:include filename="$(find ur10e_arm_with_lift)/urdf/inc/ur_transmissions.xacro" />
   <xacro:include filename="$(find ur10e_arm_with_lift)/urdf/inc/ur_common.xacro" />
-  <xacro:macro name="ur10e_with_lift_robot" params="
+  <xacro:macro name="ur_robot" params="
     name
     tf_prefix
@@ -55,5 +55,5 @@
       <xacro:include filename="$(find ur10e_arm_with_lift)/urdf/ur10e_with_lift.ros2_control.xacro" />
       <!-- ros2 control instance -->
-      <xacro:ur10e_with_lift_ros2_control
+      <xacro:ur_ros2_control
         name="${name}"
         use_fake_hardware="${use_fake_hardware}"
