Commit message: change

File: urdf/inc/ur_with_lift_transmissions.xacro (robot description, xacro)
@@ -10,5 +10,5 @@
       <type>transmission_interface/SimpleTransmission</type>
       <joint name="${prefix}lift_joint">
-        <hardwareInterface>${hw_interface}</hardwareInterface>
+        <command_interface>position</command_interface>
       </joint>
       <actuator name="{prefix}lift_motor">

File: urdf/ur10e_with_lift_macro.xacro (robot description, xacro)
@@ -1,5 +1,5 @@
 <?xml version="1.0"?>
 <robot xmlns:xacro="http://wiki.ros.org/xacro">
-  <xacro:include filename="$(find ur10e_arm_with_lift)/urdf/inc/ur_transmissions.xacro" />
+  <xacro:include filename="$(find ur10e_arm_with_lift)/urdf/inc/ur_with_lift_transmissions.xacro" />
   <xacro:include filename="$(find ur10e_arm_with_lift)/urdf/inc/ur_common.xacro" />
   <xacro:macro name="ur_robot" params="
@@ -302,6 +302,12 @@
       <origin xyz="0 0 0 " rpy="0 0 0" />
       <axis xyz="0 0 1" />
-      <limit lower="0.0" upper="1.0" effort="500" velocity="0.5"/>
-    </joint>
+      <limit lower="0.0" upper="1.0" effort="1000" velocity="10"/>
+    </joint>
+    <gazebo reference="lift_joint">
+      <kp>200.0</kp>
+      <kd>20.0</kd>
+      <ki>0.0</ki>
+      <fmax>1000.0</fmax>
+    </gazebo>
     <!-- base_joint fixes base_link to the environment -->
     <joint name="${tf_prefix}base_joint" type="fixed">
